File: keyboard_seventy/keyboard_seventy.kicad_pcb (KiCad board)
At the start: 2 copper layers, 251 parts, among them J1 ISP, J2 USB_B, J3 OLED, SW1 RESET BUTTON, SW10 SW_Push, SW100 SW_Push, SW101 SW_Push, SW102 SW_Push, SW103 SW_Push, SW104 SW_Push, SW105 SW_Push, SW106 SW_Push, SW107 SW_Push, SW108 SW_Push, SW109 SW_Push, SW11 SW_Push, SW110 SW_Push, SW111 SW_Push, SW112 SW_Push, SW113 SW_Push, SW114 SW_Push, SW115 SW_Push, SW116 SW_Push, SW117 SW_Push, SW118 SW_Push, SW119 SW_Push, SW12 SW_Push, SW120 SW_Push, SW121 SW_Push, SW13 SW_Push, SW14 SW_Push, SW15 SW_Push, SW16 SW_Push, SW17 SW_Push, SW18 SW_Push, SW19 SW_Push, SW2 SW_Push, SW20 SW_Push, SW21 SW_Push, SW22 SW_Push, SW23 SW_Push, SW24 SW_Push, SW25 SW_Push, SW26 SW_Push, SW27 SW_Push, SW28 SW_Push, SW29 SW_Push, SW3 SW_Push, SW30 SW_Push, SW31 SW_Push, SW32 SW_Push, SW33 SW_Push, SW34 SW_Push, SW35 SW_Push, SW36 SW_Push, SW37 SW_Push, SW38 SW_Push, SW39 SW_Push, SW4 SW_Push, SW40 SW_Push, SW41 SW_Push, SW42 SW_Push, SW43 SW_Push, SW44 SW_Push, SW45 SW_Push, SW46 SW_Push, SW47 SW_Push, SW48 SW_Push, SW49 SW_Push, SW5 SW_Push, SW50 SW_Push, SW51 SW_Push, SW52 SW_Push, SW53 SW_Push, SW54 SW_Push, SW55 SW_Push, SW56 SW_Push, SW57 SW_Push, SW58 SW_Push, SW59 SW_Push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

Commit message: labled and arranged keys
Parts:
- moved SW121 435.7 mm to (285.8, 152.4)
- moved SW119 387.7 mm to (247.7, 152.4)
- moved SW118 373.1 mm to (228.6, 152.4)
- moved SW120 373.0 mm to (266.7, 152.4)
- moved SW106 372.1 mm to (285.8, 133.3)
- moved SW105 362.2 mm to (266.7, 133.3)
- moved SW114 361.1 mm to (152.4, 152.4)
- moved SW117 358.3 mm to (209.6, 152.4)
- moved SW104 356.6 mm to (247.7, 133.3)
- moved SW103 355.3 mm to (228.6, 133.3)
- moved SW110 351.1 mm to (76.2, 152.4)
- moved SW113 345.4 mm to (133.3, 152.4)
- moved SW116 342.4 mm to (190.5, 152.4)
- moved SW91 336.7 mm to (285.8, 114.3)
- moved SW109 333.5 mm to (57.1, 152.4)
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
Commit message: arranged and numbered diodes
Parts:
- removed the D1 at (267.1, -135.1)
- added D113: D, Diode_THT:D_A-405_P7.62mm_Horizontal, F.Cu at (98.0, 2.00)
- moved D1 303.2 mm to (14.0, -33.0)
- moved D92 293.3 mm to (26.0, -3.00)
- moved D17 293.2 mm to (26.0, -28.0)
- moved D61 282.5 mm to (14.0, -13.0)
- moved D110 282.1 mm to (62.0, 2.00)
- moved D47 281.9 mm to (26.0, -18.0)
- moved D76 274.6 mm to (14.0, -8.00)
- moved D82 265.7 mm to (86.0, -8.00)
- moved D4 263.4 mm to (50.0, -33.0)
- moved D62 257.8 mm to (26.0, -13.0)
- moved D107 252.7 mm to (26.0, 2.00)
- moved D68 247.1 mm to (98.0, -13.0)
- moved D78 246.3 mm to (38.0, -8.00)
- moved D19 246.0 mm to (50.0, -28.0)
- moved D34 235.9 mm to (50.0, -23.0)
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- renumbered D113 to D1
Connections:
- D1 pad 1: COL8 -> COL1
- D1 pad 2: Net-(D113-Pad2) -> Net-(D1-Pad2)

Commit message: board outline and component placement
Parts:
- moved R1 7.62 mm to (276.0, -8.00)
- moved R2 7.62 mm to (273.0, -14.0)
- moved J2 4.47 mm to (283.0, -21.0)
- moved U1 2.00 mm to (211.0, -13.0)
- moved Y1 1.00 mm to (213.0, 0.00)
Other:
- board outline added: 286 x 198 mm
Changed lines of the file:
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@@
   (general
     (thickness 1.6)
-    (drawings 0)
+    (drawings 6)
     (tracks 0)
     (zones 0)
@@
   )
   (module Crystal:Resonator-3Pin_W10.0mm_H5.0mm (layer F.Cu)
-    (at 213 1 180)
+    (at 213 0 180)
     (descr "Ceramic Resomator/Filter 10.0x5.0mm^2 RedFrequency MG/MT/MX series, http://www.red-frequency.com/download/datenblatt/redfrequency-datenblatt-ir-zta.pdf, length*width=10.0x5.0mm^2 package, package length=10.0mm, package width=5.0mm, 3 pins")
     (tags "THT ceramic resonator filter")
@@
   )
   (module Package_QFP:TQFP-44_10x10mm_P0.8mm (layer F.Cu)
-    (at 211 -11)
+    (at 211 -13)
     (descr "44-Lead Plastic Thin Quad Flatpack (PT) - 10x10x1.0 mm Body [TQFP] (see Microchip Packaging Specification 00000049BS.pdf)")
     (tags "QFP 0.8")
@@
   )
   (module Resistor_THT:R_Axial_DIN0207_L6.3mm_D2.5mm_P10.16mm_Horizontal (layer F.Cu)
-    (at 270 -7)
+    (at 273 -14)
     (descr "Resistor, Axial_DIN0207 series, Axial, Horizontal, pin pitch=10.16mm, 0.25W = 1/4W, length*diameter=6.3*2.5mm^2, http://cdn-reichelt.de/documents/datenblatt/B400/1_4W%23YAG.pdf")
     (tags "Resistor Axial_DIN0207 series Axial Horizontal pin pitch 10.16mm 0.25W = 1/4W length 6.3mm diameter 2.5mm")
@@
   )
   (module Resistor_THT:R_Axial_DIN0207_L6.3mm_D2.5mm_P10.16mm_Horizontal (layer F.Cu)
-    (at 273 -1)
+    (at 276 -8)
     (descr "Resistor, Axial_DIN0207 series, Axial, Horizontal, pin pitch=10.16mm, 0.25W = 1/4W, length*diameter=6.3*2.5mm^2, http://cdn-reichelt.de/documents/datenblatt/B400/1_4W%23YAG.pdf")
     (tags "Resistor Axial_DIN0207 series Axial Horizontal pin pitch 10.16mm 0.25W = 1/4W length 6.3mm diameter 2.5mm")
@@
   )
   (module Connector_USB:USB_B_OST_USB-B1HSxx_Horizontal (layer F.Cu)
-    (at 281 -17 90)
+    (at 283 -21 90)
     (descr "USB B receptacle, Horizontal, through-hole, http://www.on-shore.com/wp-content/uploads/2015/09/usb-b1hsxx.pdf")
     (tags "USB-B receptacle horizontal through-hole")
@@
     )
   )
+  (gr_line (start 294 -37) (end 294 -36) (layer Edge.Cuts) (width 0.05))
+  (gr_line (start 8 -37) (end 294 -37) (layer Edge.Cuts) (width 0.05))
+  (gr_line (start 8 -36) (end 8 -37) (layer Edge.Cuts) (width 0.05))
+  (gr_line (start 8 161) (end 8 -36) (layer Edge.Cuts) (width 0.05))
+  (gr_line (start 294 161) (end 8 161) (layer Edge.Cuts) (width 0.05))
+  (gr_line (start 294 161) (end 294 -36) (layer Edge.Cuts) (width 0.05))
 )

Commit message: smd diodes and some routing
Parts:
- D1, D10, D100, D101, D102, D103, D104, D105, D106, D107, D108, D109, D11, D110, D111, D112, D113, D114, D115, D116, D117, D118, D119, D12, D120, D13, D14, D15, D16, D17, D18, D19, D2, D20, D21, D22, D23, D24, D25, D26, D27, D28, D29, D3, D30, D31, D32, D33, D34, D35, D36, D37, D38, D39, D4, D40, D41, D42, D43, D44, D45, D46, D47, D48, D49, D5, D50, D51, D52, D53, D54, D55, D56, D57, D58, D59, D6, D60, D61, D62, D63, D64, D65, D66, D67, D68, D69, D7, D70, D71, D72, D73, D74, D75, D76, D77, D78, D79, D8, D80, D81, D82, D83, D84, D85, D86, D87, D88, D89, D9, D90, D91, D92, D93, D94, D95, D96, D97, D98, D99: footprint Diode_THT:D_A-405_P7.62mm_Horizontal -> Diode_SMD:D_0805_2012Metric; moved to B.Cu
- moved D120 176.8 mm to (276.7, 151.3), turned to 270 degrees
- moved D119 173.2 mm to (257.6, 151.3), turned to 270 degrees
- moved D118 169.7 mm to (238.6, 151.3), turned to 270 degrees
- moved D117 166.5 mm to (219.6, 151.3), turned to 270 degrees
- moved D105 165.1 mm to (276.7, 132.3), turned to 270 degrees
- moved D116 163.5 mm to (200.5, 151.3), turned to 270 degrees
- moved D104 161.2 mm to (257.6, 132.3), turned to 270 degrees
- moved D115 160.7 mm to (181.4, 151.3), turned to 270 degrees
- moved D114 158.3 mm to (162.4, 151.3), turned to 270 degrees
- moved D103 157.5 mm to (238.6, 132.3), turned to 270 degrees
- moved D113 156.1 mm to (143.3, 151.3), turned to 270 degrees
- moved D112 154.2 mm to (124.3, 151.3), turned to 270 degrees
- moved D102 154.0 mm to (219.6, 132.3), turned to 270 degrees
- moved D90 153.8 mm to (276.7, 113.2), turned to 270 degrees
- moved D111 152.6 mm to (105.2, 151.3), turned to 270 degrees
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Other:
- board size 286 x 198 mm -> 286 x 173 mm

Commit message: wired though should check connecting gnds
Routing:
- net ROW4: track 0.00 -> 584.6 mm, vias 0 -> 7
- net ROW7: track 0.00 -> 557.6 mm, vias 0 -> 3
- net ROW3: track 0.00 -> 556.3 mm, vias 0 -> 8
- net ROW2: track 0.00 -> 530.9 mm, vias 0 -> 8
- net ROW6: track 0.00 -> 504.0 mm, vias 0 -> 8
- net ROW5: track 0.00 -> 496.2 mm, vias 0 -> 8
- net ROW8: track 0.00 -> 454.9 mm, vias 0 -> 1
- net ROW1: track 0.00 -> 440.4 mm, vias 0 -> 1
- net COL2: track 0.00 -> 368.3 mm, vias 0 -> 1
- net COL1: track 0.00 -> 330.9 mm, vias 0 -> 1
- net COL4: track 0.00 -> 320.7 mm, vias 0 -> 1
- net COL6: track 0.00 -> 297.1 mm, vias 0 -> 1
- net COL3: track 0.00 -> 283.0 mm, vias 0 -> 1
- net COL15: track 0.00 -> 279.0 mm, vias 0 -> 1
- net COL9: track 0.00 -> 267.0 mm, vias 0 -> 1
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